File: pcb/tube.kicad_sch (KiCad schematic)
At the start: 79 parts, among them J1 Screw_Terminal_01x02, J10 LED_[5..8], J11 LED_[1..4], J2 Screw_Terminal_01x02, J3 Screw_Terminal_01x02, J4 Conn_01x04_Pin, J5 Conn_01x08_Pin, J6 Conn_01x05_Pin, U1 INA226, U10 74LS32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

Commit message: PCB: Use 3.3V For Temperature Probes
Connections:
- net +3.3V: now also U6.3 (V_{DD}), U7.3 (V_{DD}), U8.3 (V_{DD})
- net +5V: no longer U6.3 (V_{DD}), U7.3 (V_{DD}), U8.3 (V_{DD})
Changed lines of the file:
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@@
+    )
+  )
+  (symbol (lib_id "power:+3.3V") (at 186.69 148.59 0) (unit 1)
+    (in_bom yes) (on_board yes) (dnp no)
+    (property "Reference" "#PWR028" (at 186.69 152.4 0)
+      (effects (font (size 1.27 1.27)) hide)
+    )
+    (property "Value" "+3.3V" (at 186.69 144.78 0)
+      (effects (font (size 1.27 1.27)))
+    )
+    (property "Footprint" "" (at 186.69 148.59 0)
+      (effects (font (size 1.27 1.27)) hide)
+    )
+    (property "Datasheet" "" (at 186.69 148.59 0)
+      (effects (font (size 1.27 1.27)) hide)
+    )
+    (pin "1")
+    (instances
+      (project "tube"
+        (path "/17a681e7-f555-4501-b0f6-333651e2bfd6"
+          (reference "#PWR028") (unit 1)
+        )
+      )
     )
   )
@@
         (path "/17a681e7-f555-4501-b0f6-333651e2bfd6"
           (reference "J10") (unit 1)
-        )
-      )
-    )
-  )
-  (symbol (lib_id "power:+5V") (at 186.69 179.07 0) (unit 1)
-    (in_bom yes) (on_board yes) (dnp no)
-    (property "Reference" "#PWR038" (at 186.69 182.88 0)
-      (effects (font (size 1.27 1.27)) hide)
-    )
-    (property "Value" "+5V" (at 186.69 176.53 90)
-      (effects (font (size 1.27 1.27)) (justify left))
-    )
-    (property "Footprint" "" (at 186.69 179.07 0)
-      (effects (font (size 1.27 1.27)) hide)
-    )
-    (property "Datasheet" "" (at 186.69 179.07 0)
-      (effects (font (size 1.27 1.27)) hide)
-    )
-    (pin "1")
-    (instances
-      (project "tube"
-        (path "/17a681e7-f555-4501-b0f6-333651e2bfd6"
-          (reference "#PWR038") (unit 1)
         )
       )
@@
     )
   )
+  (symbol (lib_id "power:+3.3V") (at 186.69 179.07 0) (unit 1)
+    (in_bom yes) (on_board yes) (dnp no)
+    (property "Reference" "#PWR038" (at 186.69 182.88 0)
+      (effects (font (size 1.27 1.27)) hide)
+    )
+    (property "Value" "+3.3V" (at 186.69 175.26 0)
+      (effects (font (size 1.27 1.27)))
+    )
+    (property "Footprint" "" (at 186.69 179.07 0)
+      (effects (font (size 1.27 1.27)) hide)
+    )
+    (property "Datasheet" "" (at 186.69 179.07 0)
+      (effects (font (size 1.27 1.27)) hide)
+    )
+    (pin "1")
+    (instances
+      (project "tube"
+        (path "/17a681e7-f555-4501-b0f6-333651e2bfd6"
+          (reference "#PWR038") (unit 1)
+        )
+      )
+    )
+  )
   (symbol (lib_id "power:+5V") (at 19.05 203.2 0) (unit 1)
     (in_bom yes) (on_board yes) (dnp no)
@@
         (path "/17a681e7-f555-4501-b0f6-333651e2bfd6"
           (reference "R11") (unit 1)
-        )
-      )
-    )
-  )
-  (symbol (lib_id "power:+5V") (at 186.69 148.59 0) (unit 1)
-    (in_bom yes) (on_board yes) (dnp no)
-    (property "Reference" "#PWR033" (at 186.69 152.4 0)
-      (effects (font (size 1.27 1.27)) hide)
-    )
-    (property "Value" "+5V" (at 186.69 146.05 90)
-      (effects (font (size 1.27 1.27)) (justify left))
-    )
-    (property "Footprint" "" (at 186.69 148.59 0)
-      (effects (font (size 1.27 1.27)) hide)
-    )
-    (property "Datasheet" "" (at 186.69 148.59 0)
-      (effects (font (size 1.27 1.27)) hide)
-    )
-    (pin "1")
-    (instances
-      (project "tube"
-        (path "/17a681e7-f555-4501-b0f6-333651e2bfd6"
-          (reference "#PWR033") (unit 1)
         )
       )
@@
     )
   )
-  (symbol (lib_id "power:+5V") (at 186.69 118.11 0) (unit 1)
-    (in_bom yes) (on_board yes) (dnp no)
-    (property "Reference" "#PWR028" (at 186.69 121.92 0)
-      (effects (font (size 1.27 1.27)) hide)
-    )
-    (property "Value" "+5V" (at 186.69 115.57 90)
-      (effects (font (size 1.27 1.27)) (justify left))
-    )
-    (property "Footprint" "" (at 186.69 118.11 0)
-      (effects (font (size 1.27 1.27)) hide)
-    )
-    (property "Datasheet" "" (at 186.69 118.11 0)
-      (effects (font (size 1.27 1.27)) hide)
-    )
-    (pin "1")
-    (instances
-      (project "tube"
-        (path "/17a681e7-f555-4501-b0f6-333651e2bfd6"
-          (reference "#PWR028") (unit 1)
-        )
-      )
-    )
-  )
   (symbol (lib_id "Mechanical:MountingHole_Pad") (at 165.1 25.4 180) (unit 1)
     (in_bom yes) (on_board yes) (dnp no) (fields_autoplaced)
@@
         )
       )
+    )
+  )
+  (symbol (lib_id "power:+3.3V") (at 186.69 118.11 0) (unit 1)
+    (in_bom yes) (on_board yes) (dnp no)
+    (property "Reference" "#PWR033" (at 186.69 121.92 0)
+      (effects (font (size 1.27 1.27)) hide)
+    )
+    (property "Value" "+3.3V" (at 186.69 114.3 0)
+      (effects (font (size 1.27 1.27)))
+    )
+    (property "Footprint" "" (at 186.69 118.11 0)
+      (effects (font (size 1.27 1.27)) hide)
+    )
+    (property "Datasheet" "" (at 186.69 118.11 0)
+      (effects (font (size 1.27 1.27)) hide)
+    )
+    (pin "1")
+    (instances
+      (project "tube"
+        (path "/17a681e7-f555-4501-b0f6-333651e2bfd6"
+          (reference "#PWR033") (unit 1)
+        )
+      )
